File: pic_proto/pic_proto1/pic_proto1.kicad_pcb (KiCad board)
At the start: 2 copper layers, 94 x 31.8 mm, 11 parts, among them J1 Conn_01x04_Male, J2 Conn_01x11, SW1 Switch_SW_SPST, U1 PIC16F84A-XXP, X1 XTAL

Commit message: Updates
Parts:
- removed the REF** at (125.7, 48.3)
- added REF**: PinHeader_1x10_P2.54mm_Vertical, Connector_PinHeader_2.54mm:PinHeader_1x10_P2.54mm_Vertical, F.Cu at (137.2, 50.8)
- added REF**: PinHeader_1x10_P2.54mm_Vertical, Connector_PinHeader_2.54mm:PinHeader_1x10_P2.54mm_Vertical, F.Cu at (134.6, 50.8)
- added REF**: PinHeader_1x10_P2.54mm_Vertical, Connector_PinHeader_2.54mm:PinHeader_1x10_P2.54mm_Vertical, F.Cu at (132.1, 50.8)
- added REF**: PinHeader_1x10_P2.54mm_Vertical, Connector_PinHeader_2.54mm:PinHeader_1x10_P2.54mm_Vertical, F.Cu at (129.5, 50.8)
- added REF**: PinHeader_1x10_P2.54mm_Vertical, Connector_PinHeader_2.54mm:PinHeader_1x10_P2.54mm_Vertical, F.Cu at (127.0, 50.8)
- added REF**: PinHeader_1x10_P2.54mm_Vertical, Connector_PinHeader_2.54mm:PinHeader_1x10_P2.54mm_Vertical, F.Cu at (124.5, 50.8)
Routing:
- net (no net): vias 423 -> 0
Other:
- board text added: "+5V"
- board text added: "GND"
- board text added: "PIC Prototype PCB V2.0 Dec 2022 menadue@gmail.com"
