File: pic_proto/pic_proto1/pic_proto1.sch (KiCad schematic (older format))
At the start: 10 parts, among them J1 Conn_01x04_Male, J2 Conn_01x11, SW1 Switch_SW_SPST, U1 PIC16F84A-XXP, X1 XTAL

Commit message: Updates
Parts:
- X1: symbol Microtan_exp:XTAL -> pic_proto1-rescue:XTAL-Microtan_exp
Changed lines of the file:
@@
 $EndComp
 $Comp
-L Microtan_65_CPU-cache:GND #PWR0101
+L pic_proto1-rescue:GND-Microtan_65_CPU-cache #PWR0101
 U 1 1 5F285E70
 P 4400 4750
@@
 	3250 2750 3700 2750
 $Comp
-L Microtan_exp:XTAL X1
+L pic_proto1-rescue:XTAL-Microtan_exp X1
 U 1 1 5F28862C
 P 2500 2950
@@
 Connection ~ 2100 3150
 $Comp
-L Microtan_65_CPU-cache:GND #PWR0104
+L pic_proto1-rescue:GND-Microtan_65_CPU-cache #PWR0104
 U 1 1 5F28B3EE
 P 2100 3650
@@
 $EndComp
 $Comp
-L Microtan_65_CPU-cache:GND #PWR0105
+L pic_proto1-rescue:GND-Microtan_65_CPU-cache #PWR0105
 U 1 1 5F28B927
 P 2750 3650
